File: blinkenkringel.sch (EAGLE design)
At the start: 84 parts, among them Q1 IRLML2502, Q2 BC337-40, Q3 BC337-40, Q4 BC337-40, Q5 BC337-40

Commit message: forgotten connection led-resistor added
Connections:
- new net N$49: LED1B.C, R38.2
- new net N$50: LED1A.C, R39.2
Changed lines of the file:
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@@
+</segment>
+</net>
+<net name="N$49" class="0">
+<segment>
+<pinref part="LED1" gate="B" pin="C"/>
+<pinref part="R38" gate="G$1" pin="2"/>
+<wire x1="93.98" y1="63.5" x2="96.52" y2="63.5" width="0.1524" layer="91"/>
+</segment>
+</net>
+<net name="N$50" class="0">
+<segment>
+<pinref part="R39" gate="G$1" pin="2"/>
+<pinref part="LED1" gate="A" pin="C"/>
+<wire x1="96.52" y1="55.88" x2="93.98" y2="55.88" width="0.1524" layer="91"/>
 </segment>
 </net>

Commit message: changed voltage divider
Parts:
- R1: value 15k -> 12k
- R2: value 33k -> 15k
Other:
- note added: "ca 1.1V Bandgap BAT LOW 2V (2x1V) max 118µA@3.2V"
- note removed: "ca 1.1V Bandgap BAT LOW 1,6V (2x0,8V) max 66µA@3.2V"
Changed lines of the file:
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@@
 <part name="BAT+" library="solpad" deviceset="MCS10B" device=""/>
 <part name="BAT-" library="solpad" deviceset="MCS10B" device=""/>
-<part name="R1" library="rcl" deviceset="R-EU_" device="0207/7" value="15k"/>
-<part name="R2" library="rcl" deviceset="R-EU_" device="0207/7" value="33k"/>
+<part name="R1" library="rcl" deviceset="R-EU_" device="0207/7" value="12k"/>
+<part name="R2" library="rcl" deviceset="R-EU_" device="0207/7" value="15k"/>
 <part name="C1" library="rcl" deviceset="CPOL-EU" device="E5-8.5" value="470u"/>
 <part name="C2" library="rcl" deviceset="CPOL-EU" device="E5-8.5" value="470u"/>
@@
 <plain>
 <text x="30.48" y="119.38" size="1.778" layer="97">ca 1.1V Bandgap
-BAT LOW 1,6V (2x0,8V)
-max 66µA@3.2V</text>
+BAT LOW 2V (2x1V)
+max 118µA@3.2V</text>
 <wire x1="45.72" y1="165.1" x2="45.72" y2="147.32" width="0.3048" layer="97"/>
 <wire x1="45.72" y1="147.32" x2="71.12" y2="147.32" width="0.3048" layer="97"/>

Commit message: capacitor at reset line for BOD detection/reset
Parts:
- added C4: 100n, rcl:C-EU025-024X044
Connections:
- net GND: now also C4.2
- net N$1: now also C4.1
Other:
- note added: "needed for clean startup after BOD"
Changed lines of the file:
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@@
 <part name="SUPPLY17" library="supply2" deviceset="GND" device=""/>
 <part name="C3" library="rcl" deviceset="C-EU" device="025-024X044" value="100n"/>
+<part name="C4" library="rcl" deviceset="C-EU" device="025-024X044" value="100n"/>
+<part name="SUPPLY18" library="supply2" deviceset="GND" device=""/>
 </parts>
 <sheets>
@@
 <text x="50.292" y="154.432" size="1.778" layer="97">DC-DC CONV
 9-4V -&gt; 5V</text>
+<text x="30.48" y="86.36" size="1.778" layer="97" rot="R180">needed for clean
+startup after BOD</text>
 </plain>
 <instances>
@@
 <instance part="SUPPLY17" gate="GND" x="96.52" y="35.56"/>
 <instance part="C3" gate="G$1" x="25.4" y="50.8"/>
+<instance part="C4" gate="G$1" x="30.48" y="88.9"/>
+<instance part="SUPPLY18" gate="GND" x="30.48" y="81.28"/>
 </instances>
 <busses>
@@
 <pinref part="SUPPLY17" gate="GND" pin="GND"/>
 <wire x1="96.52" y1="40.64" x2="96.52" y2="38.1" width="0.1524" layer="91"/>
+</segment>
+<segment>
+<pinref part="C4" gate="G$1" pin="2"/>
+<pinref part="SUPPLY18" gate="GND" pin="GND"/>
 </segment>
 </net>
@@
 <wire x1="30.48" y1="91.44" x2="33.02" y2="91.44" width="0.1524" layer="91"/>
 <pinref part="U$1" gate="G$1" pin="PA2(/RESET)"/>
-</segment>
-</net>
+<pinref part="C4" gate="G$1" pin="1"/>
+<junction x="30.48" y="91.44"/>
+</segment>
+</net>
